Commit message: Update robot.xacro

File: robot_description/urdf/robot.xacro (robot description, xacro)
@@ -66,5 +66,5 @@
 <link name="lidar_1">
   <inertial>
-    <origin xyz="1.4148987538217285e-07 0.07500008440088982 0.02500004084516777" rpy="0 0 0"/>
+    <origin xyz="1.4148987538217285e-07 0.07500008440088982 0.22500004084516777" rpy="0 0 0"/>
     <mass value="0.26554311904467726"/>
     <inertia ixx="0.000137" iyy="0.000137" izz="0.000163" ixy="-0.0" iyz="0.0" ixz="0.0"/>

Commit message: Update robot.xacro

File: robot_description/urdf/robot.xacro (robot description, xacro)
@@ -66,5 +66,5 @@
 <link name="lidar_1">
   <inertial>
-    <origin xyz="1.4148987538217285e-07 0.07500008440088982 0.22500004084516777" rpy="0 0 0"/>
+    <origin xyz="1.4148987538217285e-07 0.07500008440088982 0.02500004084516777" rpy="0 0 0"/>
     <mass value="0.26554311904467726"/>
     <inertia ixx="0.000137" iyy="0.000137" izz="0.000163" ixy="-0.0" iyz="0.0" ixz="0.0"/>
